Commit message: feat(hexo): update robot joint limits and velocities
- Integrated a new USD model (bw_modify_joint_limit/bw.usd) for the Hexo robot.
- Increased joint velocity limits for multiple joints in the URDF.
- Modified the upper limit of the right ankle pitch joint.
- Disabled the safety controller in the URDF.
- These adjustments provide the robot with a wider range of motion and faster dynamics, improving its capabilities within the simulation.

File: source/isaaclab_tasks/isaaclab_tasks/direct/humanoid_amp/motions/robot_description/bw/urdf/bw.urdf (robot description, URDF)
Before this commit: robot BwRobot, 13 links, 12 joints
Joints:
- joint right_ankle_pitch_joint: limit lower=-0.87267 upper=0.7 effort=100 velocity=40 -> lower=-0.87267 upper=0.5236 effort=100 velocity=40
- joint right_knee_joint: limit lower=-0.01 upper=1 effort=200 velocity=20 -> lower=-0.01 upper=1 effort=200 velocity=40
- joint right_leg_pitch_joint: limit lower=-1.57 upper=1.31 effort=300 velocity=32 -> lower=-1.57 upper=1.31 effort=300 velocity=40
- joint right_leg_roll_joint: limit lower=-2.9671 upper=0.5236 effort=200 velocity=20 -> lower=-2.9671 upper=0.5236 effort=200 velocity=40
- joint right_leg_yaw_joint: limit lower=-2.7576 upper=2.7576 effort=200 velocity=12 -> lower=-2.7576 upper=2.7576 effort=200 velocity=40
